File: 4004Peripheral.kicad_pcb (KiCad board)
At the start: 2 copper layers, 95.1 x 72.1 mm, 304 parts, among them J1 BUS, J2 VCC, J3 GND, J4 OUTPUT, J5 IO_IN, J6 IO_OUT, J7 SW LEVEL, J8 IO, SW0 SW0, SW1 SW1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

Commit message: SW位置入れ替え
Parts:
- added REF**: VIA-0.8-Hole-0.4mm, cd_device:VIA-0.8-Hole-0.4mm, F.Cu at (186.7, 127.4)
- added REF**: VIA-0.8-Hole-0.4mm, cd_device:VIA-0.8-Hole-0.4mm, F.Cu at (166.0, 130.0)
- moved R12 36.2 mm to (177.9, 138.8)
- moved R9 36.1 mm to (141.7, 138.6)
- moved SW0 35.8 mm to (180.6, 134.9)
- moved SW3 35.8 mm to (144.8, 134.9)
- moved R1 31.6 mm to (147.2, 132.5), turned to 180 degrees
- moved R4 29.5 mm to (177.8, 134.0)
- moved R2 18.8 mm to (154.2, 133.7)
- moved R11 12.1 mm to (166.0, 138.4)
- moved R10 11.9 mm to (154.2, 138.7)
- moved SW1 11.9 mm to (168.7, 134.9)
- moved SW2 11.9 mm to (156.7, 134.9)
- moved R3 11.8 mm to (166.0, 133.7)
- moved REF** 0.13 mm to (182.9, 132.2)
Routing:
- net Net-(J8-Pad1): track 109.0 -> 64.7 mm
- net Net-(J8-Pad4): track 71.3 -> 103.6 mm
- net Net-(J8-Pad2): track 101.5 -> 88.7 mm
- net Net-(J8-Pad3): track 82.1 -> 86.9 mm
- net VCC: track 189.9 -> 191.5 mm
Other:
- board text added: "2018-11-01"
- board text removed: "2018-05-17"

Commit message: ROMサイズ選択追加
Parts:
- added J9: ROM SIZE, Jumper:SolderJumper-3_P1.3mm_Open_RoundedPad1.0x1.5mm_NumberLabels, B.Cu at (138.5, 131.9)
- added REF**: VIA-0.8-Hole-0.4mm, cd_device:VIA-0.8-Hole-0.4mm, F.Cu at (138.9, 127.7)
- added REF**: VIA-0.8-Hole-0.4mm, cd_device:VIA-0.8-Hole-0.4mm, F.Cu at (135.2, 94.5)
- added REF**: VIA-0.8-Hole-0.4mm, cd_device:VIA-0.8-Hole-0.4mm, F.Cu at (142.3, 97.6)
- added REF**: VIA-0.8-Hole-0.4mm, cd_device:VIA-0.8-Hole-0.4mm, F.Cu at (152.4, 97.5)
- added REF**: VIA-0.8-Hole-0.4mm, cd_device:VIA-0.8-Hole-0.4mm, F.Cu at (153.6, 94.4)
- J7: footprint Connect:GS3 -> Jumper:SolderJumper-3_P1.3mm_Open_RoundedPad1.0x1.5mm_NumberLabels
- R1, R2, R3, R4: value 10k -> 3.3k
- U2: value 2716 -> 2716/2732
- moved REF** 1.58 mm to (133.6, 133.2)
- moved REF** 1.15 mm to (152.6, 128.6)
- turned J7 to 180 degrees
Connections:
- U1 pad 34: Net-(U1-Pad34) -> /A11
- U2 pad 21: VCC -> Net-(J9-Pad2)
Routing:
- net /A11: track 0.00 -> 68.5 mm
- net Net-(J9-Pad2): track 0.00 -> 43.9 mm, vias 0 -> 1
- net GND: track 12.1 -> 22.5 mm
- net VCC: track 191.5 -> 201.5 mm
- net Net-(J8-Pad2): track 88.7 -> 82.4 mm
- net Net-(J7-Pad2): track 89.5 -> 88.4 mm
Other:
- board text added: "2021-02-18"
- board text added: "2716"
- board text added: "2732"
- board text removed: "2018-11-01"

Commit message: minor silk change
Parts:
- J9: value ROM SIZE -> ROM VPP/A11
Other:
- board text added: "+5V"
- board text added: "A11"
- board text removed: "2716"
- board text removed: "2732"
